File: sheets/prog-voltage-ref.kicad_sch (KiCad schematic)
At the start: 6 parts, among them U6 MCP4726A0T-E/CH

Commit message: Use kicad footprints
Parts:
- U6: footprint Passive:SOT-23-6_L2.9-W1.6-P0.95-LS2.8-BL -> Package_TO_SOT_SMD:SOT-23-6
Changed lines of the file:
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@@
 			)
 		)
-		(property "Footprint" "Passive:SOT-23-6_L2.9-W1.6-P0.95-LS2.8-BL"
+		(property "Footprint" "Package_TO_SOT_SMD:SOT-23-6"
 			(at 95.25 72.39 0)
 			(effects

Commit message: add MCU + output
Parts:
- renumbered C22 to C17, C21 to C18, C20 to C19, R27 to R26, R28 to R27, U6 to U5
Changed lines of the file:
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@@
 		(dnp no)
 		(fields_autoplaced yes)
-		(property "Reference" "C21"
+		(property "Reference" "C18"
 			(at 81.28 71.1199 0)
 			(effects
@@
 			(project "esp32-didatic-kit"
 				(path "/f57920a5-fee7-4fe5-a133-e8b36941a5a6/68eb6d36-2b61-4a79-8b9e-43cc2ec0c3c5/714c46cd-cf03-4397-8fcb-987cad3389f9"
-					(reference "C21")
+					(reference "C18")
 					(unit 1)
 				)
@@
 		(dnp no)
 		(fields_autoplaced yes)
-		(property "Reference" "C22"
+		(property "Reference" "C17"
 			(at 68.58 71.1199 0)
 			(effects
@@
 			(project "esp32-didatic-kit"
 				(path "/f57920a5-fee7-4fe5-a133-e8b36941a5a6/68eb6d36-2b61-4a79-8b9e-43cc2ec0c3c5/714c46cd-cf03-4397-8fcb-987cad3389f9"
-					(reference "C22")
+					(reference "C17")
 					(unit 1)
 				)
@@
 		(dnp no)
 		(fields_autoplaced yes)
-		(property "Reference" "R28"
+		(property "Reference" "R27"
 			(at 139.7 72.3899 0)
 			(effects
@@
 			(project "esp32-didatic-kit"
 				(path "/f57920a5-fee7-4fe5-a133-e8b36941a5a6/68eb6d36-2b61-4a79-8b9e-43cc2ec0c3c5/714c46cd-cf03-4397-8fcb-987cad3389f9"
-					(reference "R28")
+					(reference "R27")
 					(unit 1)
 				)
@@
 		(dnp no)
 		(fields_autoplaced yes)
-		(property "Reference" "R27"
+		(property "Reference" "R26"
 			(at 139.7 58.4199 0)
 			(effects
@@
 			(project ""
 				(path "/f57920a5-fee7-4fe5-a133-e8b36941a5a6/68eb6d36-2b61-4a79-8b9e-43cc2ec0c3c5/714c46cd-cf03-4397-8fcb-987cad3389f9"
-					(reference "R27")
+					(reference "R26")
 					(unit 1)
 				)
@@
 		(dnp no)
 		(fields_autoplaced yes)
-		(property "Reference" "C20"
+		(property "Reference" "C19"
 			(at 151.13 72.3899 0)
 			(effects
@@
 			(project ""
 				(path "/f57920a5-fee7-4fe5-a133-e8b36941a5a6/68eb6d36-2b61-4a79-8b9e-43cc2ec0c3c5/714c46cd-cf03-4397-8fcb-987cad3389f9"
-					(reference "C20")
+					(reference "C19")
 					(unit 1)
 				)
@@
 		(dnp no)
 		(fields_autoplaced yes)
-		(property "Reference" "#PWR016"
+		(property "Reference" "#PWR017"
 			(at 113.03 88.9 0)
 			(effects
@@
 			(project ""
 				(path "/f57920a5-fee7-4fe5-a133-e8b36941a5a6/68eb6d36-2b61-4a79-8b9e-43cc2ec0c3c5/714c46cd-cf03-4397-8fcb-987cad3389f9"
-					(reference "#PWR016")
+					(reference "#PWR017")
 					(unit 1)
 				)
@@
 		(dnp no)
 		(fields_autoplaced yes)
-		(property "Reference" "U6"
+		(property "Reference" "U5"
 			(at 95.25 44.45 0)
 			(effects
@@
 			(project ""
 				(path "/f57920a5-fee7-4fe5-a133-e8b36941a5a6/68eb6d36-2b61-4a79-8b9e-43cc2ec0c3c5/714c46cd-cf03-4397-8fcb-987cad3389f9"
-					(reference "U6")
-					(unit 1)
-				)
+					(reference "U5")
+					(unit 1)
+				)

Commit message: Updated MCU to MCU module + set SMD comp. footprints
Parts:
- C17, C18, C19: footprint (none) -> Capacitor_SMD:C_0603_1608Metric
- R26, R27: footprint (none) -> Resistor_SMD:R_0603_1608Metric
Changed lines of the file:
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@@
 			)
 		)
-		(property "Footprint" ""
+		(property "Footprint" "Capacitor_SMD:C_0603_1608Metric"
 			(at 78.4352 76.2 0)
 			(effects
@@
 			)
 		)
-		(property "Footprint" ""
+		(property "Footprint" "Capacitor_SMD:C_0603_1608Metric"
 			(at 65.7352 76.2 0)
 			(effects
@@
 			)
 		)
-		(property "Footprint" ""
+		(property "Footprint" "Resistor_SMD:R_0603_1608Metric"
 			(at 138.938 73.66 90)
 			(effects
@@
 			)
 		)
-		(property "Footprint" ""
+		(property "Footprint" "Resistor_SMD:R_0603_1608Metric"
 			(at 138.938 59.69 90)
 			(effects
@@
 			)
 		)
-		(property "Footprint" ""
+		(property "Footprint" "Capacitor_SMD:C_0603_1608Metric"
 			(at 148.2852 77.47 0)
 			(effects
