File: sheets/voltage-ref.kicad_sch (KiCad schematic)
At the start: 5 parts, among them U5 MCP1501-40E/SN

Commit message: Use kicad footprints
Parts:
- U5: footprint Passive:SOIC-8_L4.9-W3.9-P1.27-LS6.0-BL -> Package_SO:SOIC-8_3.9x4.9mm_P1.27mm
Changed lines of the file:
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@@
 			)
 		)
-		(property "Footprint" "Passive:SOIC-8_L4.9-W3.9-P1.27-LS6.0-BL"
+		(property "Footprint" "Package_SO:SOIC-8_3.9x4.9mm_P1.27mm"
 			(at 97.79 60.96 0)
 			(effects

Commit message: add MCU + output
Parts:
- renumbered C17 to C20, C18 to C21, C19 to C22, R26 to R28, U5 to U6
Changed lines of the file:
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@@
 		(dnp no)
 		(fields_autoplaced yes)
-		(property "Reference" "C19"
+		(property "Reference" "C22"
 			(at 151.13 59.6899 0)
 			(effects
@@
 			(project "esp32-didatic-kit"
 				(path "/f57920a5-fee7-4fe5-a133-e8b36941a5a6/68eb6d36-2b61-4a79-8b9e-43cc2ec0c3c5/aea191e3-b773-40f6-a9d4-aec24cc2a210"
-					(reference "C19")
+					(reference "C22")
 					(unit 1)
 				)
@@
 		(dnp no)
 		(fields_autoplaced yes)
-		(property "Reference" "#PWR014"
+		(property "Reference" "#PWR018"
 			(at 63.5 87.63 0)
 			(effects
@@
 			(project ""
 				(path "/f57920a5-fee7-4fe5-a133-e8b36941a5a6/68eb6d36-2b61-4a79-8b9e-43cc2ec0c3c5/aea191e3-b773-40f6-a9d4-aec24cc2a210"
-					(reference "#PWR014")
+					(reference "#PWR018")
 					(unit 1)
 				)
@@
 		(dnp no)
 		(fields_autoplaced yes)
-		(property "Reference" "U5"
+		(property "Reference" "U6"
 			(at 97.79 38.1 0)
 			(effects
@@
 			(project ""
 				(path "/f57920a5-fee7-4fe5-a133-e8b36941a5a6/68eb6d36-2b61-4a79-8b9e-43cc2ec0c3c5/aea191e3-b773-40f6-a9d4-aec24cc2a210"
-					(reference "U5")
+					(reference "U6")
 					(unit 1)
 				)
@@
 		(dnp no)
 		(fields_autoplaced yes)
-		(property "Reference" "R26"
+		(property "Reference" "R28"
 			(at 135.89 39.37 90)
 			(effects
@@
 			(project ""
 				(path "/f57920a5-fee7-4fe5-a133-e8b36941a5a6/68eb6d36-2b61-4a79-8b9e-43cc2ec0c3c5/aea191e3-b773-40f6-a9d4-aec24cc2a210"
-					(reference "R26")
+					(reference "R28")
 					(unit 1)
 				)
@@
 		(dnp no)
 		(fields_autoplaced yes)
-		(property "Reference" "C18"
+		(property "Reference" "C21"
 			(at 128.27 58.4199 0)
 			(effects
@@
 			(project "esp32-didatic-kit"
 				(path "/f57920a5-fee7-4fe5-a133-e8b36941a5a6/68eb6d36-2b61-4a79-8b9e-43cc2ec0c3c5/aea191e3-b773-40f6-a9d4-aec24cc2a210"
-					(reference "C18")
+					(reference "C21")
 					(unit 1)
 				)
@@
 		(dnp no)
 		(fields_autoplaced yes)
-		(property "Reference" "C17"
+		(property "Reference" "C20"
 			(at 67.31 60.9599 0)
 			(effects
@@
 			(project ""
 				(path "/f57920a5-fee7-4fe5-a133-e8b36941a5a6/68eb6d36-2b61-4a79-8b9e-43cc2ec0c3c5/aea191e3-b773-40f6-a9d4-aec24cc2a210"
-					(reference "C17")
-					(unit 1)
-				)
+					(reference "C20")
+					(unit 1)
+				)

Commit message: Updated MCU to MCU module + set SMD comp. footprints
Parts:
- C20, C21, C22: footprint (none) -> Capacitor_SMD:C_0603_1608Metric
- R28: footprint (none) -> Resistor_SMD:R_0603_1608Metric
Changed lines of the file:
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@@
 			)
 		)
-		(property "Footprint" ""
+		(property "Footprint" "Capacitor_SMD:C_0603_1608Metric"
 			(at 148.2852 64.77 0)
 			(effects
@@
 			)
 		)
-		(property "Footprint" ""
+		(property "Footprint" "Resistor_SMD:R_0603_1608Metric"
 			(at 135.89 47.498 90)
 			(effects
@@
 			)
 		)
-		(property "Footprint" ""
+		(property "Footprint" "Capacitor_SMD:C_0603_1608Metric"
 			(at 125.4252 63.5 0)
 			(effects
@@
 			)
 		)
-		(property "Footprint" ""
+		(property "Footprint" "Capacitor_SMD:C_0603_1608Metric"
 			(at 64.4652 66.04 0)
 			(effects
