File: sheets/relay.kicad_sch (KiCad schematic)
At the start: 3 parts, among them K1 G2RL-1

Commit message: add mcu module + position components
Parts:
- renumbered R82 to R87

Commit message: Updated MCU to MCU module + set SMD comp. footprints
Parts:
- D25: footprint (none) -> LED_SMD:LED_0603_1608Metric
- R87: value R -> 18k; footprint (none) -> Resistor_SMD:R_0603_1608Metric
Changed lines of the file:
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@@
 			)
 		)
-		(property "Value" "R"
+		(property "Value" "18k"
 			(at 95.25 45.7199 0)
 			(effects
@@
 			)
 		)
-		(property "Footprint" ""
+		(property "Footprint" "Resistor_SMD:R_0603_1608Metric"
 			(at 90.932 44.45 90)
 			(effects
@@
 			)
 		)
-		(property "Footprint" ""
+		(property "Footprint" "LED_SMD:LED_0603_1608Metric"
 			(at 92.71 53.34 0)
 			(effects
