File: esp32-didatic-kit.kicad_pcb (KiCad board)
At the start: 2 copper layers, 266 x 220 mm, 142 parts, among them CON1 MIKROBUS_HOST_CONN, CON2 MIKROBUS_HOST_CONN, CON3 MIKROBUS_HOST_CONN, J2 Conn_02x05_Odd_Even, J3 Conn_02x05_Odd_Even, J4 Conn_02x05_Odd_Even, J5 Conn_02x05_Odd_Even, J6 USB_C_Receptacle, J8 MCU_MODULE_CONN, K1 G2RL-1, K10 G2RL-1, K11 G2RL-1, K12 G2RL-1, K13 G2RL-1, K14 G2RL-1, K15 G2RL-1, K16 G2RL-1, K2 G2RL-1, K3 G2RL-1, K4 G2RL-1, K5 G2RL-1, K6 G2RL-1, K7 G2RL-1, K8 G2RL-1, K9 G2RL-1, Q1 DMP2160UW-7, Q2 PDTC114EU,115, Q3 DMN2058U-7, Q4 DMN2058U-7, Q5 2N7002, Q7 2N7002, SW2 TDS08SGRNTU04, SW3 TDS08SGRNTU04, SW4 TDS08SGRNTU04, SW5 TDS08SGRNTU04, SW6 SW_DIP_x08, SW7 SW_DIP_x08, U1 LM2575-12BU, U10 HCPL2630SDVM, U11 HCPL2630SDVM, U12 HCPL2630SDVM, U13 HCPL2630SDVM, U14 HCPL2630SDVM, U15 HCPL2630SDVM, U16 HCPL2630SDVM, U17 PCF8574AT, U18 PCF8574AT, U19 PCF8574AT, U2 ST1S10PHR, U20 ULN2803A, U21 ULN2803A, U22 SN65HVD231, U23 USBLC6-2SC6, U24 CH340G, U3 ST1S10PHR, U4 MCP6H02T-E/SN, U5 MCP4726A0T-E/CH, U6 MCP1501-40E/SN, U7 ESP32-WROVER-B, U8 PCF8574AT, U9 HCPL2630SDVM

Commit message: Updated MCU to MCU module + set SMD comp. footprints
Parts:
- removed BOOT1, RST1: TL3342F160QG, Button_Switch_SMD:SW_SPST_TL3342
- removed C48, C49: 10nF, Capacitor_SMD:C_0603_1608Metric
- removed JP2, JP3, JP4, JP5: Jumper_3_Open, Connector_PinHeader_2.54mm:PinHeader_1x03_P2.54mm_Vertical
- removed U7: ESP32-WROVER-B, ICs:MODULE_ESP32-WROVER-B
- added C10: 1uF, Capacitor_SMD:C_0603_1608Metric, F.Cu at (403.3, 9.02)
- added C11: 22uF, Capacitor_SMD:C_0603_1608Metric, F.Cu at (403.3, 11.5)
- added C12: 22uF, Capacitor_SMD:C_0603_1608Metric, F.Cu at (403.3, 14.0)
- added C13: 22uF, Capacitor_SMD:C_0603_1608Metric, F.Cu at (403.3, 16.6)
- added C14: 100pF, Capacitor_SMD:C_0603_1608Metric, F.Cu at (409.3, 9.02)
- added C15: 0.1uF, Capacitor_SMD:C_0603_1608Metric, F.Cu at (409.3, 11.5)
- added C16: 0.1uF, Capacitor_SMD:C_0603_1608Metric, F.Cu at (409.3, 14.0)
- added C17: 0.1uF, Capacitor_SMD:C_0603_1608Metric, F.Cu at (409.3, 30.6)
- added C18: 0.1uF, Capacitor_SMD:C_0603_1608Metric, F.Cu at (409.3, 33.1)
- added C19: 0.1uF, Capacitor_SMD:C_0603_1608Metric, F.Cu at (409.3, 35.6)
- added C20: 1uF, Capacitor_SMD:C_0603_1608Metric, F.Cu at (415.3, 30.6)
- added C21: 100pF, Capacitor_SMD:C_0603_1608Metric, F.Cu at (415.3, 33.1)
- added C22: 2.2uF, Capacitor_SMD:C_0603_1608Metric, F.Cu at (415.3, 35.6)
- added C28: 0.1uF, Capacitor_SMD:C_0603_1608Metric, F.Cu at (435.4, 9.02)
- added C29: 0.1uF, Capacitor_SMD:C_0603_1608Metric, F.Cu at (429.4, 28.6)
- added C30: 0.1uF, Capacitor_SMD:C_0603_1608Metric, F.Cu at (441.4, 9.02)
- added C31: 0.1uF, Capacitor_SMD:C_0603_1608Metric, F.Cu at (435.4, 28.6)
- added C32: 0.1uF, Capacitor_SMD:C_0603_1608Metric, F.Cu at (423.4, 28.6)
- added C33: 0.1uF, Capacitor_SMD:C_0603_1608Metric, F.Cu at (441.4, 28.6)
- added C34: 0.1uF, Capacitor_SMD:C_0603_1608Metric, F.Cu at (423.4, 9.02)
- added C35: 0.1uF, Capacitor_SMD:C_0603_1608Metric, F.Cu at (429.4, 9.02)
- added C36: 0.1uF, Capacitor_SMD:C_0603_1608Metric, F.Cu at (431.6, -0.61)
- added C37: 0.1uF, Capacitor_SMD:C_0603_1608Metric, F.Cu at (431.6, 1.90)
- added C42: 0.1uF, Capacitor_SMD:C_0603_1608Metric, F.Cu at (437.6, -0.61)
- added C43: 0.1uF, Capacitor_SMD:C_0603_1608Metric, F.Cu at (437.6, 1.90)
- added C44: 0.1uF, Capacitor_SMD:C_0603_1608Metric, F.Cu at (431.6, -7.63)
- added C45: 0.1uF, Capacitor_SMD:C_0603_1608Metric, F.Cu at (431.6, -5.12)
- added C46: 22pF, Capacitor_SMD:C_0603_1608Metric, F.Cu at (437.6, -7.63)
- added C47: 22pF, Capacitor_SMD:C_0603_1608Metric, F.Cu at (437.6, -5.12)
- added C6: 1uF, Capacitor_SMD:C_0603_1608Metric, F.Cu at (397.3, 9.02)
- added C7: 22uF, Capacitor_SMD:C_0603_1608Metric, F.Cu at (397.3, 11.5)
- added C8: 22uF, Capacitor_SMD:C_0603_1608Metric, F.Cu at (397.3, 14.0)
- added C9: 22uF, Capacitor_SMD:C_0603_1608Metric, F.Cu at (397.3, 16.6)
- added D1: SS24, Diode_SMD:D_SMA, F.Cu at (372.6, 10.0)
- added D2: SS24, Diode_SMD:D_SMA, F.Cu at (372.6, 14.6)
- added D25: LED, LED_SMD:LED_0603_1608Metric, F.Cu at (390.7, 33.9)
- added D26: LED, LED_SMD:LED_0603_1608Metric, F.Cu at (437.7, -36.0)
- added D27: LED, LED_SMD:LED_0603_1608Metric, F.Cu at (443.7, -36.0)
- added D28: LED, LED_SMD:LED_0603_1608Metric, F.Cu at (384.7, 33.9)
- added D29: LED, LED_SMD:LED_0603_1608Metric, F.Cu at (431.6, -28.9)
- added D3: SS24, Diode_SMD:D_SMA, F.Cu at (372.6, 19.1)
- added D30: LED, LED_SMD:LED_0603_1608Metric, F.Cu at (390.7, 41.0)
- added D31: LED, LED_SMD:LED_0603_1608Metric, F.Cu at (384.7, 41.0)
- added D32: LED, LED_SMD:LED_0603_1608Metric, F.Cu at (431.6, -36.0)
- added D33: LED, LED_SMD:LED_0603_1608Metric, F.Cu at (437.7, -28.9)
- added D34: LED, LED_SMD:LED_0603_1608Metric, F.Cu at (443.7, -21.8)
- added D35: LED, LED_SMD:LED_0603_1608Metric, F.Cu at (437.7, -14.7)
- added D36: LED, LED_SMD:LED_0603_1608Metric, F.Cu at (431.6, -21.8)
- added D37: LED, LED_SMD:LED_0603_1608Metric, F.Cu at (431.6, -14.7)
- added D38: LED, LED_SMD:LED_0603_1608Metric, F.Cu at (443.7, -14.7)
- added D39: LED, LED_SMD:LED_0603_1608Metric, F.Cu at (443.7, -28.9)
- added D4: SS24, Diode_SMD:D_SMA, F.Cu at (411.4, 25.1)
- added D40: LED, LED_SMD:LED_0603_1608Metric, F.Cu at (437.7, -21.8)
- added D5: SS24, Diode_SMD:D_SMA, F.Cu at (372.6, 23.7)
- added J1: Power Input, TerminalBlock_Phoenix:TerminalBlock_Phoenix_MKDS-1,5-2-5.08_1x02_P5.08mm_Horizontal, F.Cu at (380.2, 24.7)
- added R1: 1.2k, Resistor_SMD:R_0603_1608Metric, F.Cu at (370.5, 33.8)
- added R10: 30k, Resistor_SMD:R_0603_1608Metric, F.Cu at (403.3, 24.1)
- added R100: 18k, Resistor_SMD:R_0603_1608Metric, F.Cu at (443.7, -12.1)
- added R101: 18k, Resistor_SMD:R_0603_1608Metric, F.Cu at (443.7, -26.3)
- added R102: 18k, Resistor_SMD:R_0603_1608Metric, F.Cu at (437.6, -19.2)
- added R11: 20k, Resistor_SMD:R_0603_1608Metric, F.Cu at (403.3, 26.6)
- added R12: 22K, Resistor_SMD:R_0603_1608Metric, F.Cu at (409.3, 16.6)
- added R13: 27K, Resistor_SMD:R_0603_1608Metric, F.Cu at (409.3, 19.1)
- added R14: 100k, Resistor_SMD:R_0603_1608Metric, F.Cu at (409.3, 21.6)
- added R15: 1k, Resistor_SMD:R_0603_1608Metric, F.Cu at (413.3, 9.02)
- added R16: 3.3k, Resistor_SMD:R_0603_1608Metric, F.Cu at (413.3, 11.5)
- added R17: 1k, Resistor_SMD:R_0603_1608Metric, F.Cu at (413.3, 14.0)
- added R18: 10k, Resistor_SMD:R_0603_1608Metric, F.Cu at (413.3, 16.6)
- added R19: 10k, Resistor_SMD:R_0603_1608Metric, F.Cu at (413.3, 19.1)
- added R2: 510, Resistor_SMD:R_0603_1608Metric, F.Cu at (370.5, 36.4)
- added R20: 470R, Resistor_SMD:R_0603_1608Metric, F.Cu at (413.3, 21.6)
- added R21: 10k, Resistor_SMD:R_0603_1608Metric, F.Cu at (417.4, 9.02)
- added R22: 100R, Resistor_SMD:R_0603_1608Metric, F.Cu at (417.4, 11.5)
- added R23: 10k, Resistor_SMD:R_0603_1608Metric, F.Cu at (417.4, 14.0)
- added R24: 10k, Resistor_SMD:R_0603_1608Metric, F.Cu at (417.4, 16.6)
- added R25: 10k, Resistor_SMD:R_0603_1608Metric, F.Cu at (417.4, 19.1)
- added R26: 10k, Resistor_SMD:R_0603_1608Metric, F.Cu at (409.3, 38.2)
- added R27: 10k, Resistor_SMD:R_0603_1608Metric, F.Cu at (409.3, 40.7)
- added R28: 10R, Resistor_SMD:R_0603_1608Metric, F.Cu at (415.3, 38.2)
- added R3: 10k, Resistor_SMD:R_0603_1608Metric, F.Cu at (370.5, 38.9)
- added R39: 10k, Resistor_SMD:R_0603_1608Metric, F.Cu at (435.4, 11.5)
- added R4: 10k, Resistor_SMD:R_0603_1608Metric, F.Cu at (397.3, 19.1)
- added R40: 10k, Resistor_SMD:R_0603_1608Metric, F.Cu at (435.4, 14.0)
- added R41: 390R, Resistor_SMD:R_0603_1608Metric, F.Cu at (435.4, 16.6)
- added R42: 390R, Resistor_SMD:R_0603_1608Metric, F.Cu at (435.4, 19.1)
- added R43: 100k, Resistor_SMD:R_0603_1608Metric, F.Cu at (435.4, 21.6)
- added R44: 100k, Resistor_SMD:R_0603_1608Metric, F.Cu at (435.4, 24.1)
- added R45: 10k, Resistor_SMD:R_0603_1608Metric, F.Cu at (429.4, 31.1)
- added R46: 10k, Resistor_SMD:R_0603_1608Metric, F.Cu at (429.4, 33.6)
- added R47: 390R, Resistor_SMD:R_0603_1608Metric, F.Cu at (429.4, 36.1)
- added R48: 390R, Resistor_SMD:R_0603_1608Metric, F.Cu at (429.4, 38.6)
- added R49: 100k, Resistor_SMD:R_0603_1608Metric, F.Cu at (429.4, 41.1)
- added R5: 4.7k, Resistor_SMD:R_0603_1608Metric, F.Cu at (397.3, 21.6)
- added R50: 100k, Resistor_SMD:R_0603_1608Metric, F.Cu at (429.4, 43.6)
- added R51: 10k, Resistor_SMD:R_0603_1608Metric, F.Cu at (441.4, 11.5)
- added R52: 10k, Resistor_SMD:R_0603_1608Metric, F.Cu at (441.4, 14.0)
- added R53: 390R, Resistor_SMD:R_0603_1608Metric, F.Cu at (441.4, 16.6)
- added R54: 390R, Resistor_SMD:R_0603_1608Metric, F.Cu at (441.4, 19.1)
- added R55: 100k, Resistor_SMD:R_0603_1608Metric, F.Cu at (441.4, 21.6)
- added R56: 100k, Resistor_SMD:R_0603_1608Metric, F.Cu at (441.4, 24.1)
- added R57: 10k, Resistor_SMD:R_0603_1608Metric, F.Cu at (435.4, 31.1)
- added R58: 10k, Resistor_SMD:R_0603_1608Metric, F.Cu at (435.4, 33.6)
- added R59: 390R, Resistor_SMD:R_0603_1608Metric, F.Cu at (435.4, 36.1)
- added R6: 100k, Resistor_SMD:R_0603_1608Metric, F.Cu at (397.3, 24.1)
- added R60: 390R, Resistor_SMD:R_0603_1608Metric, F.Cu at (435.4, 38.6)
- added R61: 100k, Resistor_SMD:R_0603_1608Metric, F.Cu at (435.4, 41.1)
- added R62: 100k, Resistor_SMD:R_0603_1608Metric, F.Cu at (435.4, 43.6)
- added R63: 10k, Resistor_SMD:R_0603_1608Metric, F.Cu at (423.4, 31.1)
- added R64: 10k, Resistor_SMD:R_0603_1608Metric, F.Cu at (423.4, 33.6)
- added R65: 390R, Resistor_SMD:R_0603_1608Metric, F.Cu at (423.4, 36.1)
- added R66: 390R, Resistor_SMD:R_0603_1608Metric, F.Cu at (423.4, 38.6)
- added R67: 100k, Resistor_SMD:R_0603_1608Metric, F.Cu at (423.4, 41.1)
- added R68: 100k, Resistor_SMD:R_0603_1608Metric, F.Cu at (423.4, 43.6)
- added R69: 10k, Resistor_SMD:R_0603_1608Metric, F.Cu at (441.4, 31.1)
- added R7: 20k, Resistor_SMD:R_0603_1608Metric, F.Cu at (397.3, 26.6)
- added R70: 10k, Resistor_SMD:R_0603_1608Metric, F.Cu at (441.4, 33.6)
- added R71: 390R, Resistor_SMD:R_0603_1608Metric, F.Cu at (441.4, 36.1)
- added R72: 390R, Resistor_SMD:R_0603_1608Metric, F.Cu at (441.4, 38.6)
- added R73: 100k, Resistor_SMD:R_0603_1608Metric, F.Cu at (441.4, 41.1)
- added R74: 100k, Resistor_SMD:R_0603_1608Metric, F.Cu at (441.4, 43.6)
- added R75: 10k, Resistor_SMD:R_0603_1608Metric, F.Cu at (423.4, 11.5)
- added R76: 10k, Resistor_SMD:R_0603_1608Metric, F.Cu at (423.4, 14.0)
- added R77: 390R, Resistor_SMD:R_0603_1608Metric, F.Cu at (423.4, 16.6)
- added R78: 390R, Resistor_SMD:R_0603_1608Metric, F.Cu at (423.4, 19.1)
- added R79: 100k, Resistor_SMD:R_0603_1608Metric, F.Cu at (423.4, 21.6)
- added R8: 10k, Resistor_SMD:R_0603_1608Metric, F.Cu at (403.3, 19.1)
- added R80: 100k, Resistor_SMD:R_0603_1608Metric, F.Cu at (423.4, 24.1)
- added R81: 10k, Resistor_SMD:R_0603_1608Metric, F.Cu at (429.4, 11.5)
- added R82: 10k, Resistor_SMD:R_0603_1608Metric, F.Cu at (429.4, 14.0)
- added R83: 390R, Resistor_SMD:R_0603_1608Metric, F.Cu at (429.4, 16.6)
- added R84: 390R, Resistor_SMD:R_0603_1608Metric, F.Cu at (429.4, 19.1)
- added R85: 100k, Resistor_SMD:R_0603_1608Metric, F.Cu at (429.4, 21.6)
- added R86: 100k, Resistor_SMD:R_0603_1608Metric, F.Cu at (429.4, 24.1)
- added R87: 18k, Resistor_SMD:R_0603_1608Metric, F.Cu at (390.7, 36.4)
- added R88: 18k, Resistor_SMD:R_0603_1608Metric, F.Cu at (437.6, -33.4)
- added R89: 18k, Resistor_SMD:R_0603_1608Metric, F.Cu at (443.7, -33.4)
- added R9: 30k, Resistor_SMD:R_0603_1608Metric, F.Cu at (403.3, 21.6)
- added R90: 18k, Resistor_SMD:R_0603_1608Metric, F.Cu at (384.6, 36.4)
- added R91: 18k, Resistor_SMD:R_0603_1608Metric, F.Cu at (431.6, -26.3)
- added R92: 18k, Resistor_SMD:R_0603_1608Metric, F.Cu at (390.7, 43.5)
- added R93: 18k, Resistor_SMD:R_0603_1608Metric, F.Cu at (384.6, 43.5)
- added R94: 18k, Resistor_SMD:R_0603_1608Metric, F.Cu at (431.6, -33.4)
- added R95: 18k, Resistor_SMD:R_0603_1608Metric, F.Cu at (437.6, -26.3)
- added R96: 18k, Resistor_SMD:R_0603_1608Metric, F.Cu at (443.7, -19.2)
- added R97: 18k, Resistor_SMD:R_0603_1608Metric, F.Cu at (437.6, -12.1)
- added R98: 18k, Resistor_SMD:R_0603_1608Metric, F.Cu at (431.6, -19.2)
- added R99: 18k, Resistor_SMD:R_0603_1608Metric, F.Cu at (431.6, -12.1)
- added SW8: SS-12D10L5, Connectors:SW-TH_SS-12D10L5, F.Cu at (385.0, 13.1)
- added Y3: 12MHz, Crystal:Crystal_SMD_3225-4Pin_3.2x2.5mm, F.Cu at (442.2, -6.61)
- D8: value LL4148 -> SS24; footprint Diode_SMD:D_MiniMELF -> Diode_SMD:D_SMA
- moved D8 120.9 mm to (376.6, 34.9)
- moved J8 1.00 mm to (209.3, 135.4)
Connections:
- net /IO/Output PortC/COMM0 renamed /IO/OutputE/COMM0
- net /IO/Output PortC/COMM1 renamed /IO/OutputE/COMM1
- net /IO/Output PortC/NC0 renamed /IO/OutputE/NC0
- net /IO/Output PortC/NC1 renamed /IO/OutputE/NC1
- net /IO/Output PortC/NC2 renamed /IO/OutputE/NC2
- net /IO/Output PortC/NC3 renamed /IO/OutputE/NC3
- net /IO/Output PortC/NC4 renamed /IO/OutputE/NC4
- net /IO/Output PortC/NC5 renamed /IO/OutputE/NC5
- net /IO/Output PortC/NC6 renamed /IO/OutputE/NC6
- net /IO/Output PortC/NC7 renamed /IO/OutputE/NC7
- net /IO/Output PortC/NO0 renamed /IO/OutputE/NO0
- net /IO/Output PortC/NO1 renamed /IO/OutputE/NO1
- net /IO/Output PortC/NO2 renamed /IO/OutputE/NO2
- net /IO/Output PortC/NO3 renamed /IO/OutputE/NO3
- net /IO/Output PortC/NO5 renamed /IO/OutputE/NO5
- net /IO/Output PortC/NO6 renamed /IO/OutputE/NO6
- net /IO/Output PortC/NO7 renamed /IO/OutputE/NO7
- net /IO/Output PortC/OUT0 renamed /IO/OutputE/OUT0
- net /IO/Output PortC/OUT1 renamed /IO/OutputE/OUT1
- net /IO/Output PortC/OUT2 renamed /IO/OutputE/OUT2
- net /IO/Output PortC/OUT3 renamed /IO/OutputE/OUT3
- net /IO/Output PortC/OUT4 renamed /IO/OutputE/OUT4
- net /IO/Output PortC/OUT5 renamed /IO/OutputE/OUT5
- net /IO/Output PortC/OUT6 renamed /IO/OutputE/OUT6
- net /IO/Output PortC/OUT7 renamed /IO/OutputE/OUT7
- net /IO/Output PortC/REL0 renamed /IO/OutputE/REL0
- net /IO/Output PortC/REL1 renamed /IO/OutputE/REL1
- net /IO/Output PortC/REL2 renamed /IO/OutputE/REL2
- net /IO/Output PortC/REL3 renamed /IO/OutputE/REL3
- net /IO/Output PortC/REL4 renamed /IO/OutputE/REL4
- net /IO/Output PortC/REL5 renamed /IO/OutputE/REL5
- net /IO/Output PortC/REL6 renamed /IO/OutputE/REL6
- net /IO/Output PortC/REL7 renamed /IO/OutputE/REL7
- net /IO/Output PortC/Relay Circuit1/COMM renamed /IO/OutputE/Relay Circuit1/COMM
- net /IO/Output PortC/Relay Circuit6/COMM renamed /IO/OutputE/Relay Circuit6/COMM
- net /IO/Output PortD/COMM0 renamed /IO/OutputF/COMM0
- net /IO/Output PortD/COMM1 renamed /IO/OutputF/COMM1
- net /IO/Output PortD/NC0 renamed /IO/OutputF/NC0
- net /IO/Output PortD/NC1 renamed /IO/OutputF/NC1
- net /IO/Output PortD/NC2 renamed /IO/OutputF/NC2
- net /IO/Output PortD/NC3 renamed /IO/OutputF/NC3
- net /IO/Output PortD/NC4 renamed /IO/OutputF/NC4
- net /IO/Output PortD/NC5 renamed /IO/OutputF/NC5
- net /IO/Output PortD/NC6 renamed /IO/OutputF/NC6
- net /IO/Output PortD/NC7 renamed /IO/OutputF/NC7
- net /IO/Output PortD/NO0 renamed /IO/OutputF/NO0
- net /IO/Output PortD/NO1 renamed /IO/OutputF/NO1
- net /IO/Output PortD/NO2 renamed /IO/OutputF/NO2
- net /IO/Output PortD/NO3 renamed /IO/OutputF/NO3
- net /IO/Output PortD/NO5 renamed /IO/OutputF/NO5
- net /IO/Output PortD/NO6 renamed /IO/OutputF/NO6
- net /IO/Output PortD/NO7 renamed /IO/OutputF/NO7
- net /IO/Output PortD/OUT0 renamed /IO/OutputF/OUT0
- net /IO/Output PortD/OUT1 renamed /IO/OutputF/OUT1
- net /IO/Output PortD/OUT2 renamed /IO/OutputF/OUT2
- net /IO/Output PortD/OUT3 renamed /IO/OutputF/OUT3
- net /IO/Output PortD/OUT4 renamed /IO/OutputF/OUT4
- net /IO/Output PortD/OUT5 renamed /IO/OutputF/OUT5
- net /IO/Output PortD/OUT6 renamed /IO/OutputF/OUT6
- net /IO/Output PortD/OUT7 renamed /IO/OutputF/OUT7
- net /IO/Output PortD/REL0 renamed /IO/OutputF/REL0
- net /IO/Output PortD/REL1 renamed /IO/OutputF/REL1
- net /IO/Output PortD/REL2 renamed /IO/OutputF/REL2
- net /IO/Output PortD/REL3 renamed /IO/OutputF/REL3
- net /IO/Output PortD/REL4 renamed /IO/OutputF/REL4
- net /IO/Output PortD/REL5 renamed /IO/OutputF/REL5
- net /IO/Output PortD/REL6 renamed /IO/OutputF/REL6
- net /IO/Output PortD/REL7 renamed /IO/OutputF/REL7
- net /IO/Output PortD/Relay Circuit1/COMM renamed /IO/OutputF/Relay Circuit1/COMM
- net /IO/Output PortD/Relay Circuit6/COMM renamed /IO/OutputF/Relay Circuit6/COMM
- net /Power Supply/Buck 12V/Vin renamed /Power Supply/Vraw
- C4 pad 1: /Power Supply/Buck 12V/Vout -> +12V
- C5 pad 1: /Power Supply/Buck 12V/Vout -> +12V
- D8 pad 1: /USB-SERIAL/DBG_UART.DTR -> Net-(D8-K)
- D8 pad 2: Net-(D8-A) -> +5V
- J2 pad 1: /IO/IO PortA/P0 -> /IO/IO PortC/P0
- J2 pad 2: /IO/IO PortA/P1 -> /IO/IO PortC/P1
- J2 pad 3: /IO/IO PortA/P2 -> /IO/IO PortC/P2
- J2 pad 4: /IO/IO PortA/P3 -> /IO/IO PortC/P3
- J2 pad 5: /IO/IO PortA/P4 -> /IO/IO PortC/P4
- J2 pad 6: /IO/IO PortA/P5 -> /IO/IO PortC/P5
- J2 pad 7: /IO/IO PortA/P6 -> /IO/IO PortC/P6
- J2 pad 8: /IO/IO PortA/P7 -> /IO/IO PortC/P7
- J3 pad 1: /IO/IO PortB/P0 -> /IO/IO PortD/P0
- J3 pad 2: /IO/IO PortB/P1 -> /IO/IO PortD/P1
- J3 pad 3: /IO/IO PortB/P2 -> /IO/IO PortD/P2
- J3 pad 4: /IO/IO PortB/P3 -> /IO/IO PortD/P3
- J3 pad 5: /IO/IO PortB/P4 -> /IO/IO PortD/P4
- J3 pad 6: /IO/IO PortB/P5 -> /IO/IO PortD/P5
- J3 pad 7: /IO/IO PortB/P6 -> /IO/IO PortD/P6
- J3 pad 8: /IO/IO PortB/P7 -> /IO/IO PortD/P7
- J4 pad 1: /IO/IO PortC/P0 -> /IO/IO PortE/P0
- J4 pad 2: /IO/IO PortC/P1 -> /IO/IO PortE/P1
- J4 pad 3: /IO/IO PortC/P2 -> /IO/IO PortE/P2
- J4 pad 4: /IO/IO PortC/P3 -> /IO/IO PortE/P3
- J4 pad 5: /IO/IO PortC/P4 -> /IO/IO PortE/P4
- J4 pad 6: /IO/IO PortC/P5 -> /IO/IO PortE/P5
- J4 pad 7: /IO/IO PortC/P6 -> /IO/IO PortE/P6
- J4 pad 8: /IO/IO PortC/P7 -> /IO/IO PortE/P7
- J5 pad 1: /IO/IO PortD/P0 -> /IO/IO PortF/P0
- J5 pad 2: /IO/IO PortD/P1 -> /IO/IO PortF/P1
- J5 pad 3: /IO/IO PortD/P2 -> /IO/IO PortF/P2
- J5 pad 4: /IO/IO PortD/P3 -> /IO/IO PortF/P3
- J5 pad 5: /IO/IO PortD/P4 -> /IO/IO PortF/P4
- J5 pad 6: /IO/IO PortD/P5 -> /IO/IO PortF/P5
- J5 pad 7: /IO/IO PortD/P6 -> /IO/IO PortF/P6
- J5 pad 8: /IO/IO PortD/P7 -> /IO/IO PortF/P7
- J8 pad 1: unconnected-(J8A-Pin_1-Pad1) -> +5V
- J8 pad 10: unconnected-(J8A-Pin_10-Pad10) -> +5V
- J8 pad 11: unconnected-(J8A-Pin_11-Pad11) -> /MCU/HSPI.SCK
- J8 pad 12: unconnected-(J8A-Pin_12-Pad12) -> +5V
- J8 pad 13: unconnected-(J8A-Pin_13-Pad13) -> /MCU/HSPI.MISO
- J8 pad 14: unconnected-(J8A-Pin_14-Pad14) -> +5V
- J8 pad 15: unconnected-(J8A-Pin_15-Pad15) -> /MCU/HSPI.MOSI
- J8 pad 16: unconnected-(J8A-Pin_16-Pad16) -> +5V
- J8 pad 17: unconnected-(J8A-Pin_17-Pad17) -> /MCU/HSPI.CS
- J8 pad 18: unconnected-(J8A-Pin_18-Pad18) -> +5V
- J8 pad 19: unconnected-(J8A-Pin_19-Pad19) -> /MCU/GPI.34
- J8 pad 2: unconnected-(J8A-Pin_2-Pad2) -> +5V
- J8 pad 20: unconnected-(J8A-Pin_20-Pad20) -> +5V
- J8 pad 21: unconnected-(J8A-Pin_21-Pad21) -> /MCU/GPI.35
- J8 pad 22: unconnected-(J8A-Pin_22-Pad22) -> +5V
- J8 pad 23: unconnected-(J8A-Pin_23-Pad23) -> /MCU/GPI.36
- J8 pad 24: unconnected-(J8A-Pin_24-Pad24) -> +5V
- J8 pad 25: unconnected-(J8A-Pin_25-Pad25) -> /MCU/GPI.39
- J8 pad 26: unconnected-(J8A-Pin_26-Pad26) -> +5V
- J8 pad 28: unconnected-(J8A-Pin_28-Pad28) -> +5V
- J8 pad 3: unconnected-(J8A-Pin_3-Pad3) -> /USB-SERIAL/DBG_UART.RX
- J8 pad 30: unconnected-(J8A-Pin_30-Pad30) -> +5V
- J8 pad 32: unconnected-(J8A-Pin_32-Pad32) -> +5V
- J8 pad 33: unconnected-(J8B-Pin_1-Pad33) -> /MCU/PA0
- J8 pad 34: unconnected-(J8B-Pin_2-Pad34) -> +5V
- J8 pad 35: unconnected-(J8B-Pin_3-Pad35) -> /MCU/PA1
- J8 pad 36: unconnected-(J8B-Pin_4-Pad36) -> +5V
- J8 pad 37: unconnected-(J8B-Pin_5-Pad37) -> /MCU/PA2
- J8 pad 38: unconnected-(J8B-Pin_6-Pad38) -> +5V
- J8 pad 39: unconnected-(J8B-Pin_7-Pad39) -> /MCU/PA3
- J8 pad 4: unconnected-(J8A-Pin_4-Pad4) -> +5V
- J8 pad 40: unconnected-(J8B-Pin_8-Pad40) -> +5V
- J8 pad 41: unconnected-(J8B-Pin_9-Pad41) -> /MCU/PA4
- J8 pad 42: unconnected-(J8B-Pin_10-Pad42) -> +5V
- J8 pad 43: unconnected-(J8B-Pin_11-Pad43) -> /MCU/PA5
- J8 pad 44: unconnected-(J8B-Pin_12-Pad44) -> +5V
- J8 pad 45: unconnected-(J8B-Pin_13-Pad45) -> /MCU/PA6
- J8 pad 46: unconnected-(J8B-Pin_14-Pad46) -> +5V
- J8 pad 47: unconnected-(J8B-Pin_15-Pad47) -> /MCU/PA7
- J8 pad 48: unconnected-(J8B-Pin_16-Pad48) -> +5V
- J8 pad 49: unconnected-(J8B-Pin_17-Pad49) -> /MCU/PB0
- J8 pad 5: unconnected-(J8A-Pin_5-Pad5) -> /USB-SERIAL/DBG_UART.TX
- J8 pad 50: unconnected-(J8B-Pin_18-Pad50) -> +5V
- J8 pad 51: unconnected-(J8B-Pin_19-Pad51) -> /MCU/PB1
- J8 pad 52: unconnected-(J8B-Pin_20-Pad52) -> +5V
- J8 pad 53: unconnected-(J8B-Pin_21-Pad53) -> /MCU/PB2
- J8 pad 54: unconnected-(J8B-Pin_22-Pad54) -> +5V
- J8 pad 55: unconnected-(J8B-Pin_23-Pad55) -> /MCU/PB3
- J8 pad 56: unconnected-(J8B-Pin_24-Pad56) -> +5V
- J8 pad 57: unconnected-(J8B-Pin_25-Pad57) -> /MCU/PB4
- J8 pad 58: unconnected-(J8B-Pin_26-Pad58) -> +5V
- J8 pad 59: unconnected-(J8B-Pin_27-Pad59) -> /MCU/I2C0.SDA
- J8 pad 6: unconnected-(J8A-Pin_6-Pad6) -> +5V
- J8 pad 60: unconnected-(J8B-Pin_28-Pad60) -> +5V
- J8 pad 61: unconnected-(J8B-Pin_29-Pad61) -> /MCU/PB6
- J8 pad 62: unconnected-(J8B-Pin_30-Pad62) -> +5V
- J8 pad 63: unconnected-(J8B-Pin_31-Pad63) -> /MCU/PB7
- J8 pad 64: unconnected-(J8B-Pin_32-Pad64) -> +5V
- J8 pad 65: unconnected-(J8C-Pin_1-Pad65) -> +3V3
- J8 pad 66: unconnected-(J8C-Pin_2-Pad66) -> +5V
- J8 pad 67: unconnected-(J8C-Pin_3-Pad67) -> /MCU/I2C0.SCL
- J8 pad 7: unconnected-(J8A-Pin_7-Pad7) -> /USB-SERIAL/DBG_UART.DTR
- J8 pad 70: unconnected-(J8C-Pin_6-Pad70) -> +5V
- J8 pad 71: unconnected-(J8C-Pin_7-Pad71) -> /MCU/I2C1.SCL
- J8 pad 72: unconnected-(J8C-Pin_8-Pad72) -> +5V
- J8 pad 73: unconnected-(J8C-Pin_9-Pad73) -> /MCU/I2C1.SDA
- J8 pad 74: unconnected-(J8C-Pin_10-Pad74) -> +5V
- J8 pad 75: unconnected-(J8C-Pin_11-Pad75) -> /Can Bus/CAN.TX
- J8 pad 76: unconnected-(J8C-Pin_12-Pad76) -> +5V
- J8 pad 77: unconnected-(J8C-Pin_13-Pad77) -> /Can Bus/CAN.RX
- J8 pad 78: unconnected-(J8C-Pin_14-Pad78) -> +5V
- J8 pad 79: unconnected-(J8C-Pin_15-Pad79) -> /MCU/VSPI.SCK
- J8 pad 8: unconnected-(J8A-Pin_8-Pad8) -> +5V
- J8 pad 80: unconnected-(J8C-Pin_16-Pad80) -> +5V
- J8 pad 81: unconnected-(J8C-Pin_17-Pad81) -> /MCU/VSPI.MISO
- J8 pad 82: unconnected-(J8C-Pin_18-Pad82) -> +5V
- J8 pad 83: unconnected-(J8C-Pin_19-Pad83) -> /MCU/VSPI.MOSI
- J8 pad 84: unconnected-(J8C-Pin_20-Pad84) -> +5V
- J8 pad 85: unconnected-(J8C-Pin_21-Pad85) -> /MCU/VSPI.CS0
- J8 pad 86: unconnected-(J8C-Pin_22-Pad86) -> +5V
- J8 pad 87: unconnected-(J8C-Pin_23-Pad87) -> /MCU/VSPI.CS1
- J8 pad 88: unconnected-(J8C-Pin_24-Pad88) -> +5V
- J8 pad 89: unconnected-(J8C-Pin_25-Pad89) -> /MCU/JTAG.TMS
- J8 pad 9: unconnected-(J8A-Pin_9-Pad9) -> /USB-SERIAL/DBG_UART.RTS
- J8 pad 90: unconnected-(J8C-Pin_26-Pad90) -> +5V
- J8 pad 91: unconnected-(J8C-Pin_27-Pad91) -> /MCU/JTAG.TDI
- J8 pad 92: unconnected-(J8C-Pin_28-Pad92) -> +5V
- J8 pad 93: unconnected-(J8C-Pin_29-Pad93) -> /MCU/JTAG.TCK
- J8 pad 94: unconnected-(J8C-Pin_30-Pad94) -> +5V
- J8 pad 95: unconnected-(J8C-Pin_31-Pad95) -> /MCU/JTAG.TDO
- J8 pad 96: unconnected-(J8C-Pin_32-Pad96) -> +5V
- K10 pad A1: /IO/Output PortD/Relay Circuit1/Coil -> /IO/OutputF/Relay Circuit1/Coil
- K2 pad A1: /IO/Output PortC/Relay Circuit1/Coil -> /IO/OutputE/Relay Circuit1/Coil
- L1 pad 1: Net-(D5-K) -> Net-(D8-K)
- L1 pad 2: /Power Supply/Buck 12V/Vout -> +12V
- SW2 pad 1: /IO/IO PortA/P0 -> /IO/IO PortC/P0
- SW2 pad 2: /IO/IO PortA/P1 -> /IO/IO PortC/P1
- SW2 pad 3: /IO/IO PortA/P2 -> /IO/IO PortC/P2
- SW2 pad 4: /IO/IO PortA/P3 -> /IO/IO PortC/P3
- SW2 pad 5: /IO/IO PortA/P4 -> /IO/IO PortC/P4
- SW2 pad 6: /IO/IO PortA/P5 -> /IO/IO PortC/P5
- SW2 pad 7: /IO/IO PortA/P6 -> /IO/IO PortC/P6
- SW2 pad 8: /IO/IO PortA/P7 -> /IO/IO PortC/P7
- SW3 pad 1: /IO/IO PortB/P0 -> /IO/IO PortD/P0
- SW3 pad 2: /IO/IO PortB/P1 -> /IO/IO PortD/P1
- SW3 pad 3: /IO/IO PortB/P2 -> /IO/IO PortD/P2
- SW3 pad 4: /IO/IO PortB/P3 -> /IO/IO PortD/P3
- SW3 pad 5: /IO/IO PortB/P4 -> /IO/IO PortD/P4
- SW3 pad 6: /IO/IO PortB/P5 -> /IO/IO PortD/P5
- SW3 pad 7: /IO/IO PortB/P6 -> /IO/IO PortD/P6
- SW3 pad 8: /IO/IO PortB/P7 -> /IO/IO PortD/P7
- SW4 pad 1: /IO/IO PortC/P0 -> /IO/IO PortE/P0
- SW4 pad 2: /IO/IO PortC/P1 -> /IO/IO PortE/P1
- SW4 pad 3: /IO/IO PortC/P2 -> /IO/IO PortE/P2
- SW4 pad 4: /IO/IO PortC/P3 -> /IO/IO PortE/P3
- SW4 pad 5: /IO/IO PortC/P4 -> /IO/IO PortE/P4
- SW4 pad 6: /IO/IO PortC/P5 -> /IO/IO PortE/P5
- SW4 pad 7: /IO/IO PortC/P6 -> /IO/IO PortE/P6
- SW4 pad 8: /IO/IO PortC/P7 -> /IO/IO PortE/P7
- SW5 pad 1: /IO/IO PortD/P0 -> /IO/IO PortF/P0
- SW5 pad 2: /IO/IO PortD/P1 -> /IO/IO PortF/P1
- SW5 pad 3: /IO/IO PortD/P2 -> /IO/IO PortF/P2
- SW5 pad 4: /IO/IO PortD/P3 -> /IO/IO PortF/P3
- SW5 pad 5: /IO/IO PortD/P4 -> /IO/IO PortF/P4
- SW5 pad 6: /IO/IO PortD/P5 -> /IO/IO PortF/P5
- SW5 pad 7: /IO/IO PortD/P6 -> /IO/IO PortF/P6
- SW5 pad 8: /IO/IO PortD/P7 -> /IO/IO PortF/P7
- SW6 pad 1: /IO/IO PortC/P0 -> /IO/IO PortE/P0
- SW6 pad 2: /IO/IO PortC/P1 -> /IO/IO PortE/P1
- SW6 pad 3: /IO/IO PortC/P2 -> /IO/IO PortE/P2
- SW6 pad 4: /IO/IO PortC/P3 -> /IO/IO PortE/P3
- SW6 pad 5: /IO/IO PortC/P4 -> /IO/IO PortE/P4
- SW6 pad 6: /IO/IO PortC/P5 -> /IO/IO PortE/P5
- SW6 pad 7: /IO/IO PortC/P6 -> /IO/IO PortE/P6
- SW6 pad 8: /IO/IO PortC/P7 -> /IO/IO PortE/P7
- SW7 pad 1: /IO/IO PortD/P0 -> /IO/IO PortF/P0
- SW7 pad 2: /IO/IO PortD/P1 -> /IO/IO PortF/P1
- SW7 pad 3: /IO/IO PortD/P2 -> /IO/IO PortF/P2
- SW7 pad 4: /IO/IO PortD/P3 -> /IO/IO PortF/P3
- SW7 pad 5: /IO/IO PortD/P4 -> /IO/IO PortF/P4
- SW7 pad 6: /IO/IO PortD/P5 -> /IO/IO PortF/P5
- SW7 pad 7: /IO/IO PortD/P6 -> /IO/IO PortF/P6
- SW7 pad 8: /IO/IO PortD/P7 -> /IO/IO PortF/P7
- U1 pad 2: Net-(D5-K) -> Net-(D8-K)
- U10 pad 6: /IO/IO PortA/P5 -> /IO/IO PortC/P5
- U11 pad 6: /IO/IO PortA/P3 -> /IO/IO PortC/P3
- U12 pad 6: /IO/IO PortA/P7 -> /IO/IO PortC/P7
- U13 pad 6: /IO/IO PortB/P1 -> /IO/IO PortD/P1
- U14 pad 6: /IO/IO PortB/P3 -> /IO/IO PortD/P3
- U15 pad 6: /IO/IO PortB/P5 -> /IO/IO PortD/P5
- U16 pad 6: /IO/IO PortB/P7 -> /IO/IO PortD/P7
- U17 pad 1: /IO/IO PortB/ADDR[0..2] -> /IO/IO PortD/ADDR[0..2]
- U17 pad 10: /IO/IO PortB/P5 -> /IO/IO PortD/P5
- U17 pad 11: /IO/IO PortB/P6 -> /IO/IO PortD/P6
- U17 pad 12: /IO/IO PortB/P7 -> /IO/IO PortD/P7
- U17 pad 13: /IO/IO PortB/INTR_N -> /IO/IO PortD/INTR_N
- U17 pad 2: /IO/IO PortB/ADDR[0..2] -> /IO/IO PortD/ADDR[0..2]
- U17 pad 3: /IO/IO PortB/ADDR[0..2] -> /IO/IO PortD/ADDR[0..2]
- U17 pad 4: /IO/IO PortB/P0 -> /IO/IO PortD/P0
- U17 pad 5: /IO/IO PortB/P1 -> /IO/IO PortD/P1
- U17 pad 6: /IO/IO PortB/P2 -> /IO/IO PortD/P2
- U17 pad 7: /IO/IO PortB/P3 -> /IO/IO PortD/P3
- U17 pad 9: /IO/IO PortB/P4 -> /IO/IO PortD/P4
- U18 pad 1: /IO/IO PortC/ADDR[0..2] -> /IO/IO PortE/ADDR[0..2]
- U18 pad 10: /IO/IO PortC/P5 -> /IO/IO PortE/P5
- U18 pad 11: /IO/IO PortC/P6 -> /IO/IO PortE/P6
- U18 pad 12: /IO/IO PortC/P7 -> /IO/IO PortE/P7
- U18 pad 2: /IO/IO PortC/ADDR[0..2] -> /IO/IO PortE/ADDR[0..2]
- U18 pad 3: /IO/IO PortC/ADDR[0..2] -> /IO/IO PortE/ADDR[0..2]
- U18 pad 4: /IO/IO PortC/P0 -> /IO/IO PortE/P0
- U18 pad 5: /IO/IO PortC/P1 -> /IO/IO PortE/P1
- U18 pad 6: /IO/IO PortC/P2 -> /IO/IO PortE/P2
- U18 pad 7: /IO/IO PortC/P3 -> /IO/IO PortE/P3
- U18 pad 9: /IO/IO PortC/P4 -> /IO/IO PortE/P4
- U19 pad 1: /IO/IO PortD/ADDR[0..2] -> /IO/IO PortF/ADDR[0..2]
- U19 pad 10: /IO/IO PortD/P5 -> /IO/IO PortF/P5
- U19 pad 11: /IO/IO PortD/P6 -> /IO/IO PortF/P6
- U19 pad 12: /IO/IO PortD/P7 -> /IO/IO PortF/P7
- U19 pad 13: /IO/IO PortD/INTR_N -> /IO/IO PortF/INTR_N
- U19 pad 2: /IO/IO PortD/ADDR[0..2] -> /IO/IO PortF/ADDR[0..2]
- U19 pad 3: /IO/IO PortD/ADDR[0..2] -> /IO/IO PortF/ADDR[0..2]
- U19 pad 4: /IO/IO PortD/P0 -> /IO/IO PortF/P0
- U19 pad 5: /IO/IO PortD/P1 -> /IO/IO PortF/P1
- U19 pad 6: /IO/IO PortD/P2 -> /IO/IO PortF/P2
- U19 pad 7: /IO/IO PortD/P3 -> /IO/IO PortF/P3
- U19 pad 9: /IO/IO PortD/P4 -> /IO/IO PortF/P4
- U8 pad 1: /IO/IO PortA/ADDR[0..2] -> /IO/IO PortC/ADDR[0..2]
- U8 pad 10: /IO/IO PortA/P5 -> /IO/IO PortC/P5
- U8 pad 11: /IO/IO PortA/P6 -> /IO/IO PortC/P6
- U8 pad 12: /IO/IO PortA/P7 -> /IO/IO PortC/P7
- U8 pad 2: /IO/IO PortA/ADDR[0..2] -> /IO/IO PortC/ADDR[0..2]
- U8 pad 3: /IO/IO PortA/ADDR[0..2] -> /IO/IO PortC/ADDR[0..2]
- U8 pad 4: /IO/IO PortA/P0 -> /IO/IO PortC/P0
- U8 pad 5: /IO/IO PortA/P1 -> /IO/IO PortC/P1
- U8 pad 6: /IO/IO PortA/P2 -> /IO/IO PortC/P2
- U8 pad 7: /IO/IO PortA/P3 -> /IO/IO PortC/P3
- U8 pad 9: /IO/IO PortA/P4 -> /IO/IO PortC/P4
- U9 pad 6: /IO/IO PortA/P1 -> /IO/IO PortC/P1

Commit message: add PA an PB ports
Parts:
- removed J4, J5: Conn_02x05_Odd_Even, Connector_PinHeader_2.54mm:PinHeader_2x05_P2.54mm_Vertical
- removed SW3, SW4, SW5: TDS08SGRNTU04, Connectors:TDS08SGRNTU04
- added J10: Conn_02x05_Odd_Even, Connector_PinHeader_2.54mm:PinHeader_2x05_P2.54mm_Vertical, F.Cu at (376.1, 75.7)
- added J13: Conn_02x05_Odd_Even, Connector_PinHeader_2.54mm:PinHeader_2x05_P2.54mm_Vertical, F.Cu at (552.1, 101.7)
- added J14: Conn_02x05_Odd_Even, Connector_PinHeader_2.54mm:PinHeader_2x05_P2.54mm_Vertical, F.Cu at (522.6, 84.9)
- added J15: Conn_02x05_Odd_Even, Connector_PinHeader_2.54mm:PinHeader_2x05_P2.54mm_Vertical, F.Cu at (552.1, 68.2)
- added JP10: Jumper_2_Bridged, Jumper:SolderJumper-2_P1.3mm_Bridged_RoundedPad1.0x1.5mm, F.Cu at (474.6, 176.5)
- added JP11: Jumper_2_Bridged, Jumper:SolderJumper-2_P1.3mm_Bridged_RoundedPad1.0x1.5mm, F.Cu at (474.6, 180.0)
- added JP12: Jumper_2_Bridged, Jumper:SolderJumper-2_P1.3mm_Bridged_RoundedPad1.0x1.5mm, F.Cu at (478.9, 172.9)
- added JP13: Jumper_2_Bridged, Jumper:SolderJumper-2_P1.3mm_Bridged_RoundedPad1.0x1.5mm, F.Cu at (478.9, 176.5)
- added JP14: Jumper_2_Bridged, Jumper:SolderJumper-2_P1.3mm_Bridged_RoundedPad1.0x1.5mm, F.Cu at (478.9, 180.0)
- added JP2: Jumper_2_Bridged, Jumper:SolderJumper-2_P1.3mm_Bridged_RoundedPad1.0x1.5mm, F.Cu at (465.9, 172.9)
- added JP3: Jumper_2_Bridged, Jumper:SolderJumper-2_P1.3mm_Bridged_RoundedPad1.0x1.5mm, F.Cu at (465.9, 176.5)
- added JP4: Jumper_2_Bridged, Jumper:SolderJumper-2_P1.3mm_Bridged_RoundedPad1.0x1.5mm, F.Cu at (465.9, 180.0)
- added JP5: Jumper_2_Bridged, Jumper:SolderJumper-2_P1.3mm_Bridged_RoundedPad1.0x1.5mm, F.Cu at (470.2, 172.9)
- added JP7: Jumper_2_Bridged, Jumper:SolderJumper-2_P1.3mm_Bridged_RoundedPad1.0x1.5mm, F.Cu at (470.2, 176.5)
- added JP8: Jumper_2_Bridged, Jumper:SolderJumper-2_P1.3mm_Bridged_RoundedPad1.0x1.5mm, F.Cu at (470.2, 180.0)
- added JP9: Jumper_2_Bridged, Jumper:SolderJumper-2_P1.3mm_Bridged_RoundedPad1.0x1.5mm, F.Cu at (474.6, 172.9)
- added REF**: MountingHole_4.3mm_M4, MountingHole:MountingHole_4.3mm_M4, F.Cu at (334.8, 32.9)
- added REF**: MountingHole_4.3mm_M4, MountingHole:MountingHole_4.3mm_M4, F.Cu at (83.7, 32.9)
- added REF**: MountingHole_4.3mm_M4, MountingHole:MountingHole_4.3mm_M4, F.Cu at (83.7, 238.0)
- added REF**: MountingHole_4.3mm_M4, MountingHole:MountingHole_4.3mm_M4, F.Cu at (334.8, 238.0)
- added SW1: TDS08SGRNTU04, Connectors:TDS08SGRNTU04, F.Cu at (565.0, 124.0)
- added SW10: TDS08SGRNTU04, Connectors:TDS08SGRNTU04, F.Cu at (396.2, 81.2)
- added SW13: TDS08SGRNTU04, Connectors:TDS08SGRNTU04, F.Cu at (572.1, 107.2)
- added SW14: TDS08SGRNTU04, Connectors:TDS08SGRNTU04, F.Cu at (542.6, 90.5)
- added SW15: TDS08SGRNTU04, Connectors:TDS08SGRNTU04, F.Cu at (572.1, 73.7)
- R41, R42, R47, R48, R53, R54, R59, R60, R65, R66, R71, R72, R77, R78, R83, R84: footprint Resistor_SMD:R_0603_1608Metric -> Resistor_SMD:R_1210_3225Metric
- U10, U11, U12, U13, U14, U15, U16, U9: footprint ICs:PDIP-8_L9.6-W6.4-P2.54-LS7.9-BL -> ICs:PDIP8_GW
- moved R84 324.9 mm to (105.8, 48.3), turned to -90 degrees
- moved R85 324.3 mm to (108.3, 67.1), turned to -90 degrees
- moved R82 322.8 mm to (108.4, 47.9), turned to -90 degrees
- moved R86 321.5 mm to (110.8, 67.1), turned to -90 degrees
- moved C35 321.2 mm to (113.3, 66.2)
- moved R81 320.8 mm to (110.6, 47.9), turned to 90 degrees
- moved R83 317.7 mm to (113.2, 48.3), turned to -90 degrees
- moved R72 313.6 mm to (128.0, 48.3), turned to -90 degrees
- moved R73 312.0 mm to (130.5, 67.1), turned to -90 degrees
- moved R70 311.1 mm to (130.6, 47.9), turned to -90 degrees
- moved R74 309.3 mm to (133.0, 67.1), turned to -90 degrees
- moved R69 309.0 mm to (132.8, 47.9), turned to 90 degrees
- moved C33 308.2 mm to (135.5, 66.2)
- moved R78 307.9 mm to (116.9, 48.3), turned to -90 degrees
- moved R79 307.4 mm to (119.4, 67.1), turned to -90 degrees
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Connections:
- C1 pad 2: +5V -> GND
- C10 pad 2: +5V -> GND
- C11 pad 2: +5V -> GND
- C12 pad 2: +5V -> GND
- C13 pad 2: +5V -> GND
- C15 pad 2: +5V -> GND
- C16 pad 2: +5V -> GND
- C17 pad 2: +5V -> GND
- C18 pad 2: +5V -> GND
- C19 pad 2: +5V -> GND
- C2 pad 2: +5V -> GND
- C20 pad 2: +5V -> GND
- C21 pad 2: +5V -> GND
- C22 pad 2: +5V -> GND
- C28 pad 2: +5V -> GND
- C29 pad 2: +5V -> GND
- C3 pad 2: +5V -> GND
- C30 pad 2: +5V -> GND
- C31 pad 2: +5V -> GND
- C32 pad 2: +5V -> GND
- C33 pad 2: +5V -> GND
- C34 pad 2: +5V -> GND
- C35 pad 2: +5V -> GND
- C36 pad 2: +5V -> GND
- C37 pad 2: +5V -> GND
- C38 pad 2: +5V -> GND
- C39 pad 2: +5V -> GND
- C4 pad 2: +5V -> GND
- C40 pad 2: +5V -> GND
- C41 pad 2: +5V -> GND
- C42 pad 2: +5V -> GND
- C43 pad 2: +5V -> GND
- C44 pad 2: +5V -> GND
- C45 pad 2: +5V -> GND
- C46 pad 2: +5V -> GND
- C47 pad 2: +5V -> GND
- C5 pad 2: +5V -> GND
- C6 pad 2: +5V -> GND
- C7 pad 2: +5V -> GND
- C8 pad 2: +5V -> GND
- C9 pad 2: +5V -> GND
- CON1 pad P8: +5V -> GND
- CON1 pad P9: +5V -> GND
- CON2 pad P8: +5V -> GND
- CON2 pad P9: +5V -> GND
- CON3 pad P8: +5V -> GND
- CON3 pad P9: +5V -> GND
- D1 pad 2: +5V -> GND
- D5 pad 2: +5V -> GND
- D8 pad 2: +5V -> GND
- J2 pad 1: /IO/IO PortC/P0 -> /IO/PA0
- J2 pad 10: +5V -> GND
- J2 pad 2: /IO/IO PortC/P1 -> /IO/PA1
- J2 pad 3: /IO/IO PortC/P2 -> /IO/PA2
- J2 pad 4: /IO/IO PortC/P3 -> /IO/PA3
- J2 pad 5: /IO/IO PortC/P4 -> /IO/PA4
- J2 pad 6: /IO/IO PortC/P5 -> /IO/PA5
- J2 pad 7: /IO/IO PortC/P6 -> /IO/PA6
- J2 pad 8: /IO/IO PortC/P7 -> /IO/PA7
- J3 pad 1: /IO/IO PortD/P0 -> /IO/PB0
- J3 pad 10: +5V -> GND
- J3 pad 2: /IO/IO PortD/P1 -> /IO/PB1
- J3 pad 3: /IO/IO PortD/P2 -> /IO/PB2
- J3 pad 4: /IO/IO PortD/P3 -> /IO/PB3
- J3 pad 5: /IO/IO PortD/P4 -> /IO/PB4
- J3 pad 6: /IO/IO PortD/P5 -> /IO/PB5
- J3 pad 7: /IO/IO PortD/P6 -> /IO/PB6
- J3 pad 8: /IO/IO PortD/P7 -> /IO/PB7
- J6 pad A1: +5V -> GND
- J6 pad A12: +5V -> GND
- J6 pad B1: +5V -> GND
- J6 pad B12: +5V -> GND
- J6 pad S1: +5V -> GND
- J8 pad 10: +5V -> GND
- J8 pad 12: +5V -> GND
- J8 pad 14: +5V -> GND
- J8 pad 16: +5V -> GND
- J8 pad 18: +5V -> GND
- J8 pad 2: +5V -> GND
- J8 pad 20: +5V -> GND
- J8 pad 22: +5V -> GND
- J8 pad 24: +5V -> GND
- J8 pad 26: +5V -> GND
- J8 pad 28: +5V -> GND
- J8 pad 30: +5V -> GND
- J8 pad 32: +5V -> GND
- J8 pad 33: /MCU/PA0 -> /IO/PA0
- J8 pad 34: +5V -> GND
- J8 pad 35: /MCU/PA1 -> /IO/PA1
- J8 pad 36: +5V -> GND
- J8 pad 37: /MCU/PA2 -> /IO/PA2
- J8 pad 38: +5V -> GND
- J8 pad 39: /MCU/PA3 -> /IO/PA3
- J8 pad 4: +5V -> GND
- J8 pad 40: +5V -> GND
- J8 pad 41: /MCU/PA4 -> /IO/PA4
- J8 pad 42: +5V -> GND
- J8 pad 43: /MCU/PA5 -> /IO/PA5
- J8 pad 44: +5V -> GND
- J8 pad 45: /MCU/PA6 -> /IO/PA6
- J8 pad 46: +5V -> GND
- J8 pad 47: /MCU/PA7 -> /IO/PA7
- J8 pad 48: +5V -> GND
- J8 pad 49: /MCU/PB0 -> /IO/PB0
- J8 pad 50: +5V -> GND
- J8 pad 51: /MCU/PB1 -> /IO/PB1
- J8 pad 52: +5V -> GND
- J8 pad 53: /MCU/PB2 -> /IO/PB2
- J8 pad 54: +5V -> GND
- J8 pad 55: /MCU/PB3 -> /IO/PB3
- J8 pad 56: +5V -> GND
- J8 pad 57: /MCU/PB4 -> /IO/PB4
- J8 pad 58: +5V -> GND
- J8 pad 59: /MCU/I2C0.SDA -> /IO/PB5
- J8 pad 6: +5V -> GND
- J8 pad 60: +5V -> GND
- J8 pad 61: /MCU/PB6 -> /IO/PB6
- J8 pad 62: +5V -> GND
- J8 pad 63: /MCU/PB7 -> /IO/PB7
- J8 pad 64: +5V -> GND
- J8 pad 66: +5V -> GND
- J8 pad 70: +5V -> GND
- J8 pad 72: +5V -> GND
- J8 pad 74: +5V -> GND
- J8 pad 76: +5V -> GND
- J8 pad 78: +5V -> GND
- J8 pad 8: +5V -> GND
- J8 pad 80: +5V -> GND
- J8 pad 82: +5V -> GND
- J8 pad 84: +5V -> GND
- J8 pad 86: +5V -> GND
- J8 pad 88: +5V -> GND
- J8 pad 90: +5V -> GND
- J8 pad 92: +5V -> GND
- J8 pad 94: +5V -> GND
- J8 pad 96: +5V -> GND
- JP6 pad 2: +5V -> GND
- Q2 pad 2: +5V -> GND
- Q3 pad 2: +5V -> GND
- Q4 pad 2: +5V -> GND
- R1 pad 1: +5V -> GND
- R106 pad 1: +5V -> GND
- R107 pad 2: +5V -> GND
- R11 pad 1: +5V -> GND
- R12 pad 1: +5V -> GND
- R13 pad 1: +5V -> GND
- R17 pad 2: +5V -> GND
- R21 pad 1: +5V -> GND
- R27 pad 1: +5V -> GND
- R44 pad 1: +5V -> /IO/IO PortC/P0
- R50 pad 1: +5V -> /IO/IO PortC/P4
- R56 pad 1: +5V -> /IO/IO PortC/P2
- R62 pad 1: +5V -> /IO/IO PortC/P6
- R68 pad 1: +5V -> /IO/IO PortD/P0
- R7 pad 1: +5V -> GND
- R74 pad 1: +5V -> /IO/IO PortD/P2
- R80 pad 1: +5V -> /IO/IO PortD/P4
- R86 pad 1: +5V -> /IO/IO PortD/P6
- SW2 pad 1: /IO/IO PortC/P0 -> /IO/PB0
- SW2 pad 2: /IO/IO PortC/P1 -> /IO/PB1
- SW2 pad 3: /IO/IO PortC/P2 -> /IO/PB2
- SW2 pad 4: /IO/IO PortC/P3 -> /IO/PB3
- SW2 pad 5: /IO/IO PortC/P4 -> /IO/PB4
- SW2 pad 6: /IO/IO PortC/P5 -> /IO/PB5
- SW2 pad 7: /IO/IO PortC/P6 -> /IO/PB6
- SW2 pad 8: /IO/IO PortC/P7 -> /IO/PB7
- SW2 pad 9: +5V -> GND
- TB1 pad 1: /IO/Inputs/RAW_A1 -> /IO/Inputs/RAW_A0
- TB1 pad 2: /IO/Inputs/RAW_A0 -> /IO/Inputs/RAW_A1
- TB2 pad 1: /IO/Inputs/RAW_A3 -> /IO/Inputs/RAW_A2
- TB2 pad 2: /IO/Inputs/RAW_A2 -> /IO/Inputs/RAW_A3
- TB29 pad 2: +5V -> GND
- TB3 pad 1: /IO/Inputs/RAW_A5 -> /IO/Inputs/RAW_A4
- TB3 pad 2: /IO/Inputs/RAW_A4 -> /IO/Inputs/RAW_A5
- TB30 pad 2: +5V -> GND
- TB4 pad 1: /IO/Inputs/RAW_A7 -> /IO/Inputs/RAW_A6
- TB4 pad 2: /IO/Inputs/RAW_A6 -> /IO/Inputs/RAW_A7
- TB5 pad 1: /IO/Inputs/RAW_B1 -> /IO/Inputs/RAW_B0
- TB5 pad 2: /IO/Inputs/RAW_B0 -> /IO/Inputs/RAW_B1
- TB6 pad 1: /IO/Inputs/RAW_B3 -> /IO/Inputs/RAW_B2
- TB6 pad 2: /IO/Inputs/RAW_B2 -> /IO/Inputs/RAW_B3
- TB7 pad 1: /IO/Inputs/RAW_B5 -> /IO/Inputs/RAW_B4
- TB7 pad 2: /IO/Inputs/RAW_B4 -> /IO/Inputs/RAW_B5
- TB8 pad 1: /IO/Inputs/RAW_B7 -> /IO/Inputs/RAW_B6
- TB8 pad 2: /IO/Inputs/RAW_B6 -> /IO/Inputs/RAW_B7
- U1 pad 3: +5V -> GND
- U10 pad 5: +5V -> GND
- U10 pad 7: +5V -> /IO/IO PortC/P4
- U11 pad 5: +5V -> GND
- U11 pad 7: +5V -> /IO/IO PortC/P2
- U12 pad 5: +5V -> GND
- U12 pad 7: +5V -> /IO/IO PortC/P6
- U13 pad 5: +5V -> GND
- U13 pad 7: +5V -> /IO/IO PortD/P0
- U14 pad 5: +5V -> GND
- U14 pad 7: +5V -> /IO/IO PortD/P2
- U15 pad 5: +5V -> GND
- U15 pad 7: +5V -> /IO/IO PortD/P4
- U16 pad 5: +5V -> GND
- U16 pad 7: +5V -> /IO/IO PortD/P6
- U17 pad 8: +5V -> GND
- U18 pad 8: +5V -> GND
- U19 pad 8: +5V -> GND
- U2 pad 4: +5V -> GND
- U2 pad 5: +5V -> GND
- U2 pad 8: +5V -> GND
- U2 pad 9: +5V -> GND
- U20 pad 9: +5V -> GND
- U21 pad 9: +5V -> GND
- U22 pad 2: +5V -> GND
- U23 pad 2: +5V -> GND
- U24 pad 1: +5V -> GND
- U3 pad 4: +5V -> GND
- U3 pad 5: +5V -> GND
- U3 pad 8: +5V -> GND
- U3 pad 9: +5V -> GND
- U4 pad 4: +5V -> GND
- U5 pad 2: +5V -> GND
- U6 pad 2: +5V -> GND
- U6 pad 4: +5V -> GND
- U6 pad 5: +5V -> GND
- U6 pad 6: +5V -> GND
- U8 pad 8: +5V -> GND
- U9 pad 5: +5V -> GND
- U9 pad 7: +5V -> /IO/IO PortC/P0
Other:
- outline, holes or cut-outs redrawn
- board text added: "IN_A0"
- board text added: "IN_A1"
- board text added: "IN_A2"
- board text added: "IN_A3"
- board text added: "IN_A4"
- board text added: "IN_A5"
- board text added: "IN_A6"
- board text added: "IN_A7"
- board text added: "IN_B0"
- board text added: "IN_B1"
- board text added: "IN_B2"
- board text added: "IN_B3"
- board text added: "IN_B4"
- board text added: "IN_B5"
- board text added: "IN_B6"
- board text added: "IN_B7"
- board text added: "IVCC"
